File: USB PD/CYP3177.kicad_sch (KiCad schematic)
At the start: 31 parts, among them Q301 PJD35P03, Q302 PJD35P03, Q303 NMOS, U301 CYPD3177-24LQ, U302 NCP1117-3.3_SOT223

Commit message: addaed changes to CYPD3177
Parts:
- D302: value 15V -> 18V; footprint Diode_SMD:D_SMA -> Diode_SMD:D_SOD-123; JLCPCB C442456 -> C82088; now fitted
Other:
- note added: "STM control for charging. Pullup to ensure charging even when STM is off"
- moved on the sheet: C307, C310, U302
Changed lines of the file:
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@@
 	(generator_version "10.0")
 	(paper "A4")
+	(rectangle
+		(start 87.63 87.63)
+		(end 101.6 95.25)
+		(stroke
+			(width 0)
+			(type solid)
+			(color 255 11 30 1)
+		)
+		(fill
+			(type none)
+		)
+	)
+	(rectangle
+		(start 66.04 26.67)
+		(end 81.28 35.56)
+		(stroke
+			(width 0)
+			(type solid)
+			(color 255 11 30 1)
+		)
+		(fill
+			(type none)
+		)
+	)
+	(rectangle
+		(start 143.51 46.99)
+		(end 273.05 96.52)
+		(stroke
+			(width 0)
+			(type solid)
+			(color 255 11 30 1)
+		)
+		(fill
+			(type none)
+		)
+	)
+	(rectangle
+		(start 195.58 25.4)
+		(end 207.01 48.26)
+		(stroke
+			(width 0)
+			(type solid)
+			(color 255 11 30 1)
+		)
+		(fill
+			(type none)
+		)
+	)
 	(text "VBUS_MIN, VBUS_MAX"
 		(exclude_from_sim no)
@@
 		)
 	)
+	(text "STM control for charging. \nPullup to ensure charging even when STM is off"
+		(exclude_from_sim no)
+		(at 169.164 93.218 0)
+		(effects
+			(font
+				(size 1.27 1.27)
+			)
+		)
+	)
 	(text "PULL-DOWN\n"
 		(exclude_from_sim no)
@@
 	)
 	(junction
-		(at 261.62 59.055)
+		(at 261.62 63.5)
 		(diameter 0)
 		(color 0 0 0 0)
@@
 	)
 	(junction
-		(at 245.11 75.565)
+		(at 245.11 80.01)
 		(diameter 0)
 		(color 0 0 0 0)
@@
 	)
 	(junction
-		(at 227.33 59.055)
+		(at 227.33 63.5)
 		(diameter 0)
 		(color 0 0 0 0)
@@
 	(wire
 		(pts
-			(xy 227.33 65.405) (xy 227.33 59.055)
+			(xy 227.33 69.85) (xy 227.33 63.5)
 		)
 		(stroke
@@
 	(wire
 		(pts
-			(xy 261.62 59.055) (xy 261.62 65.405)
+			(xy 261.62 63.5) (xy 261.62 69.85)
 		)
 		(stroke
@@
 	(wire
 		(pts
-			(xy 252.73 59.055) (xy 261.62 59.055)
+			(xy 252.73 63.5) (xy 261.62 63.5)
 		)
 		(stroke
@@
 	(wire
 		(pts
-			(xy 261.62 70.485) (xy 261.62 75.565)
+			(xy 261.62 74.93) (xy 261.62 80.01)
 		)
 		(stroke
@@
 	(wire
 		(pts
-			(xy 245.11 66.675) (xy 245.11 75.565)
+			(xy 245.11 71.12) (xy 245.11 80.01)
 		)
 		(stroke
@@
 	(wire
 		(pts
-			(xy 227.33 52.705) (xy 227.33 59.055)
+			(xy 227.33 57.15) (xy 227.33 63.5)
 		)
 		(stroke
@@
 	(wire
 		(pts
-			(xy 261.62 75.565) (xy 245.11 75.565)
+			(xy 261.62 80.01) (xy 245.11 80.01)
 		)
 		(stroke
@@
 	(wire
 		(pts
-			(xy 245.11 75.565) (xy 245.11 80.645)
+			(xy 245.11 80.01) (xy 245.11 85.09)
 		)
 		(stroke
@@
 	(wire
 		(pts
-			(xy 245.11 75.565) (xy 227.33 75.565)
+			(xy 245.11 80.01) (xy 227.33 80.01)
 		)
 		(stroke
@@
 	(wire
 		(pts
-			(xy 227.33 59.055) (xy 237.49 59.055)
+			(xy 227.33 63.5) (xy 237.49 63.5)
 		)
 		(stroke
@@
 	(wire
 		(pts
-			(xy 261.62 52.705) (xy 261.62 59.055)
+			(xy 261.62 57.15) (xy 261.62 63.5)
 		)
 		(stroke
@@
 	(wire
 		(pts
-			(xy 227.33 75.565) (xy 227.33 70.485)
+			(xy 227.33 80.01) (xy 227.33 74.93)
 		)
 		(stroke
@@
 	(symbol
 		(lib_id "power:+3.3V")
-		(at 261.62 52.705 0)
+		(at 261.62 57.15 0)
 		(unit 1)
 		(body_style 1)
@@
 		(fields_autoplaced yes)
 		(property "Reference" "#PWR0319"
-			(at 261.62 56.515 0)
+			(at 261.62 60.96 0)
 			(hide yes)
 			(show_name no)
@@
 		)
 		(property "Value" "+3.3V"
-			(at 261.62 47.625 0)
+			(at 261.62 52.07 0)
 			(show_name no)
 			(do_not_autoplace no)
@@
 		)
 		(property "Footprint" ""
-			(at 261.62 52.705 0)
+			(at 261.62 57.15 0)
 			(hide yes)
 			(show_name no)
@@
 		)
 		(property "Datasheet" ""
-			(at 261.62 52.705 0)
+			(at 261.62 57.15 0)
 			(hide yes)
 			(show_name no)
@@
 		)
 		(property "Description" ""
-			(at 261.62 52.705 0)
+			(at 261.62 57.15 0)
 			(show_name no)
 			(do_not_autoplace no)
@@
 		(exclude_from_sim no)
 		(in_bom yes)
-		(on_board no)
+		(on_board yes)
 		(in_pos_files yes)
-		(dnp yes)
+		(dnp no)
 		(fields_autoplaced yes)
 		(property "Reference" "D302"
@@
 			)
 		)
-		(property "Value" "15V"
+		(property "Value" "18V"
 			(at 201.93 38.0999 90)
 			(show_name no)
@@
 			)
 		)
-		(property "Footprint" "Diode_SMD:D_SMA"
+		(property "Footprint" "Diode_SMD:D_SOD-123"
 			(at 199.39 36.83 0)
 			(hide yes)
@@
 			)
 		)
-		(property "JLCPCB" "C442456"
+		(property "JLCPCB" "C82088"
 			(at 199.39 36.83 90)
 			(hide yes)
@@
 	(symbol
 		(lib_id "power:Vout")
-		(at 227.33 52.705 0)
+		(at 227.33 57.15 0)
 		(unit 1)
 		(body_style 1)
@@
 		(fields_autoplaced yes)
 		(property "Reference" "#PWR0322"
-			(at 227.33 56.515 0)
+			(at 227.33 60.96 0)
 			(hide yes)
 			(show_name no)
@@
 		)
 		(property "Value" "Vout"
-			(at 229.87 51.4349 0)
+			(at 229.87 55.8799 0)
 			(show_name no)
 			(do_not_autoplace no)
@@
 		)
 		(property "Footprint" ""
-			(at 227.33 52.705 0)
+			(at 227.33 57.15 0)
 			(hide yes)
 			(show_name no)
@@
 		)
 		(property "Datasheet" ""
-			(at 227.33 52.705 0)
+			(at 227.33 57.15 0)
 			(hide yes)
 			(show_name no)
@@
 		)
 		(property "Description" ""
-			(at 227.33 52.705 0)
+			(at 227.33 57.15 0)
 			(show_name no)
 			(do_not_autoplace no)
@@
 	(symbol
 		(lib_id "power:GND")
-		(at 245.11 80.645 0)
+		(at 245.11 85.09 0)
 		(unit 1)
 		(body_style 1)
@@
 		(fields_autoplaced yes)
 		(property "Reference" "#PWR0321"
-			(at 245.11 86.995 0)
+			(at 245.11 91.44 0)
 			(hide yes)
 			(show_name no)
@@
 		)
 		(property "Value" "GND"
-			(at 245.11 85.09 0)
+			(at 245.11 89.535 0)
 			(show_name no)
 			(do_not_autoplace no)
@@
 		)
 		(property "Footprint" ""
-			(at 245.11 80.645 0)
+			(at 245.11 85.09 0)
 			(hide yes)
 			(show_name no)
@@
 		)
 		(property "Datasheet" ""
-			(at 245.11 80.645 0)
+			(at 245.11 85.09 0)
 			(hide yes)
 			(show_name no)
@@
 		)
 		(property "Description" ""
-			(at 245.11 80.645 0)
+			(at 245.11 85.09 0)
 			(show_name no)
 			(do_not_autoplace no)
@@
 	(symbol
 		(lib_id "Regulator_Linear:NCP1117-3.3_SOT223")
-		(at 245.11 59.055 0)
+		(at 245.11 63.5 0)
 		(unit 1)
 		(body_style 1)
@@
 		(fields_autoplaced yes)
 		(property "Reference" "U302"
-			(at 245.11 52.705 0)
+			(at 245.11 57.15 0)
 			(show_name no)
 			(do_not_autoplace no)
@@
 		)
 		(property "Value" "NCP1117-3.3_SOT223"
-			(at 245.11 55.245 0)
+			(at 245.11 59.69 0)
 			(show_name no)
 			(do_not_autoplace no)
@@
 		)
 		(property "Footprint" "Package_TO_SOT_SMD:SOT-223-3_TabPin2"
-			(at 245.11 53.975 0)
+			(at 245.11 58.42 0)
 			(hide yes)
 			(show_name no)
@@
 		)
 		(property "Datasheet" "http://www.onsemi.com/pub_link/Collateral/NCP1117-D.PDF"
-			(at 247.65 65.405 0)
+			(at 247.65 69.85 0)
 			(hide yes)
 			(show_name no)
@@
 		)
 		(property "Description" "1A Low drop-out regulator, Fixed Output 3.3V, SOT-223"
-			(at 245.11 59.055 0)
+			(at 245.11 63.5 0)
 			(hide yes)
 			(show_name no)
@@
 		)
 		(property "LCSC" "C26537"
-			(at 245.11 59.055 0)
+			(at 245.11 63.5 0)
 			(hide yes)
 			(show_name no)
@@
 		)
 		(property "Field6" ""
-			(at 245.11 59.055 0)
+			(at 245.11 63.5 0)
 			(hide yes)
 			(show_name no)
@@
 	(symbol
 		(lib_id "Device:C_Small")
-		(at 227.33 67.945 0)
+		(at 227.33 72.39 0)
 		(unit 1)
 		(body_style 1)
@@
 		(fields_autoplaced yes)
 		(property "Reference" "C307"
-			(at 229.87 66.6812 0)
+			(at 229.87 71.1262 0)
 			(show_name no)
 			(do_not_autoplace no)
@@
 		)
 		(property "Value" "10u"
-			(at 229.87 69.2212 0)
+			(at 229.87 73.6662 0)
 			(show_name no)
 			(do_not_autoplace no)
@@
 		)
 		(property "Footprint" "Capacitor_SMD:C_0805_2012Metric_Pad1.18x1.45mm_HandSolder"
-			(at 227.33 67.945 0)
+			(at 227.33 72.39 0)
 			(hide yes)
 			(show_name no)
@@
 		)
 		(property "Datasheet" ""
-			(at 227.33 67.945 0)
+			(at 227.33 72.39 0)
 			(hide yes)
 			(show_name no)
@@
 		)
 		(property "Description" ""
-			(at 227.33 67.945 0)
+			(at 227.33 72.39 0)
 			(show_name no)
 			(do_not_autoplace no)
@@
 	(symbol
 		(lib_id "Device:C_Small")
-		(at 261.62 67.945 0)
+		(at 261.62 72.39 0)
 		(unit 1)
 		(body_style 1)
@@
 		(fields_autoplaced yes)
 		(property "Reference" "C310"
-			(at 264.16 66.6812 0)
+			(at 264.16 71.1262 0)
 			(show_name no)
 			(do_not_autoplace no)
@@
 		)
 		(property "Value" "10u"
-			(at 264.16 69.2212 0)
+			(at 264.16 73.6662 0)
 			(show_name no)
 			(do_not_autoplace no)
@@
 		)
 		(property "Footprint" "Capacitor_SMD:C_0805_2012Metric_Pad1.18x1.45mm_HandSolder"
-			(at 261.62 67.945 0)
+			(at 261.62 72.39 0)
 			(hide yes)
 			(show_name no)
@@
 		)
 		(property "Datasheet" ""
-			(at 261.62 67.945 0)
+			(at 261.62 72.39 0)
 			(hide yes)
 			(show_name no)
@@
 		)
 		(property "Description" ""
-			(at 261.62 67.945 0)
+			(at 261.62 72.39 0)
 			(show_name no)
 			(do_not_autoplace no)
